Commit message: Use MikataArm model

File: open_manipulator_description/urdf/open_manipulator.urdf.xacro (robot description, xacro)
@@ -31,14 +31,14 @@
   <link name="link1">
     <visual>
-      <origin xyz="0 0 0" rpy="0 0 0"/>
-      <geometry>
-        <mesh filename="package://open_manipulator_description/meshes/chain_link1.stl" scale="0.001 0.001 0.001"/>
-      </geometry>
-      <material name="grey"/>
-    </visual>
-    <collision>
-      <origin xyz="0 0 0" rpy="0 0 0"/>
-      <geometry>
-        <mesh filename="package://open_manipulator_description/meshes/chain_link1.stl" scale="0.001 0.001 0.001"/>
+      <origin xyz="0 0 0" rpy="0 0 ${-pi*0.5}"/>
+      <geometry>
+        <mesh filename="package://open_manipulator_description/meshes/chain_link1.stl"/>
+      </geometry>
+      <material name="grey"/>
+    </visual>
+    <collision>
+      <origin xyz="0 0 0" rpy="0 0 ${-pi*0.5}"/>
+      <geometry>
+        <mesh filename="package://open_manipulator_description/meshes/chain_link1.stl"/>
       </geometry>
     </collision>
@@ -62,7 +62,7 @@
     <parent link="link1"/>
     <child link="link2"/>
-    <origin xyz="0.012 0.0 0.017" rpy="0 0 0"/>
+    <origin xyz="0 0 0.0355" rpy="0 0 0"/>
     <axis xyz="0 0 1"/>
-    <limit velocity="4.8" effort="1" lower="${-pi*0.9}" upper="${pi*0.9}" />
+    <limit velocity="4.8" effort="1" lower="${-pi}" upper="${pi}" />
   </joint>
   <!-- Transmission 1 -->
@@ -71,14 +71,14 @@
   <link name="link2">
     <visual>
-      <origin xyz="0 0 0.019" rpy="0 0 0"/>
-      <geometry>
-        <mesh filename="package://open_manipulator_description/meshes/chain_link2.stl" scale="0.001 0.001 0.001"/>
-      </geometry>
-      <material name="grey"/>
-    </visual>
-    <collision>
-      <origin xyz="0 0 0.019" rpy="0 0 0"/>
-      <geometry>
-        <mesh filename="package://open_manipulator_description/meshes/chain_link2.stl" scale="0.001 0.001 0.001"/>
+      <origin xyz="0 0 0.0405" rpy="${pi*0.5} 0 ${pi*0.5}"/>
+      <geometry>
+        <mesh filename="package://open_manipulator_description/meshes/chain_link2.stl"/>
+      </geometry>
+      <material name="grey"/>
+    </visual>
+    <collision>
+      <origin xyz="0 0 0.0405" rpy="${pi*0.5} 0 ${pi*0.5}"/>
+      <geometry>
+        <mesh filename="package://open_manipulator_description/meshes/chain_link2.stl"/>
       </geometry>
     </collision>
@@ -102,7 +102,7 @@
     <parent link="link2"/>
     <child link="link3"/>
-    <origin xyz="0.0 0.0 0.0595" rpy="0 0 0"/>
+    <origin xyz="0 0 0.0405" rpy="0 0 0"/>
     <axis xyz="0 1 0"/>
-    <limit velocity="4.8" effort="1" lower="${-pi*0.57}" upper="${pi*0.5}" />
+    <limit velocity="4.8" effort="1" lower="-1.85" upper="2.07" />
   </joint>
   <!-- Transmission 2 -->
@@ -111,14 +111,14 @@
   <link name="link3">
     <visual>
-      <origin xyz="0 0 0" rpy="0 0 0"/>
-      <geometry>
-        <mesh filename="package://open_manipulator_description/meshes/chain_link3.stl" scale="0.001 0.001 0.001"/>
-      </geometry>
-      <material name="grey"/>
-    </visual>
-    <collision>
-      <origin xyz="0 0 0" rpy="0 0 0"/>
-      <geometry>
-        <mesh filename="package://open_manipulator_description/meshes/chain_link3.stl" scale="0.001 0.001 0.001"/>
+      <origin xyz="0.024 0 0.148" rpy="0 0 ${-pi*0.5}"/>
+      <geometry>
+        <mesh filename="package://open_manipulator_description/meshes/chain_link3.stl"/>
+      </geometry>
+      <material name="grey"/>
+    </visual>
+    <collision>
+      <origin xyz="0.024 0 0.148" rpy="0 0 ${-pi*0.5}"/>
+      <geometry>
+        <mesh filename="package://open_manipulator_description/meshes/chain_link3.stl"/>
       </geometry>
     </collision>
@@ -142,7 +142,7 @@
     <parent link="link3"/>
     <child link="link4"/>
-    <origin xyz="0.024 0 0.128" rpy="0 0 0"/>
+    <origin xyz="0.024 0 0.148" rpy=" 0 0 0"/>
     <axis xyz="0 1 0"/>
-    <limit velocity="4.8" effort="1" lower="${-pi*0.3}" upper="${pi*0.44}" />
+    <limit velocity="4.8" effort="1" lower="-1.85" upper="1.41" />
   </joint>
   <!-- Transmission 3 -->
@@ -151,14 +151,14 @@
   <link name="link4">
     <visual>
-      <origin xyz="0 0 0" rpy="0 0 0"/>
-      <geometry>
-        <mesh filename="package://open_manipulator_description/meshes/chain_link4.stl" scale="0.001 0.001 0.001"/>
-      </geometry>
-      <material name="grey"/>
-    </visual>
-    <collision>
-      <origin xyz="0 0 0" rpy="0 0 0"/>
-      <geometry>
-        <mesh filename="package://open_manipulator_description/meshes/chain_link4.stl" scale="0.001 0.001 0.001"/>
+      <origin xyz="0.150 0 0" rpy="0 ${pi} ${-pi*0.5}"/>
+      <geometry>
+        <mesh filename="package://open_manipulator_description/meshes/chain_link4.stl"/>
+      </geometry>
+      <material name="grey"/>
+    </visual>
+    <collision>
+      <origin xyz="0.150 0 0" rpy="0 ${pi} ${-pi*0.5}"/>
+      <geometry>
+        <mesh filename="package://open_manipulator_description/meshes/chain_link4.stl"/>
       </geometry>
     </collision>
@@ -182,7 +182,7 @@
     <parent link="link4"/>
     <child link="link5"/>
-    <origin xyz="0.124 0.0 0.0" rpy="0 0 0"/>
+    <origin xyz="0.150 0 0" rpy="0 0 0"/>
     <axis xyz="0 1 0"/>
-    <limit velocity="4.8" effort="1" lower="${-pi*0.57}" upper="${pi*0.65}" />
+    <limit velocity="4.8" effort="1" lower="-1.64" upper="1.78" />
   </joint>
   <!-- Transmission 4 -->
@@ -193,12 +193,12 @@
       <origin xyz="0 0 0" rpy="0 0 0"/>
       <geometry>
-        <mesh filename="package://open_manipulator_description/meshes/chain_link5.stl" scale="0.001 0.001 0.001"/>
-      </geometry>
-      <material name="grey"/>
-    </visual>
-    <collision>
-      <origin xyz="0 0 0" rpy="0 0 0"/>
-      <geometry>
-        <mesh filename="package://open_manipulator_description/meshes/chain_link5.stl" scale="0.001 0.001 0.001"/>
+        <mesh filename="package://open_manipulator_description/meshes/chain_link5.stl"/>
+      </geometry>
+      <material name="grey"/>
+    </visual>
+    <collision>
+      <origin xyz="0 0 0" rpy="0 0 0"/>
+      <geometry>
+        <mesh filename="package://open_manipulator_description/meshes/chain_link5.stl"/>
       </geometry>
     </collision>
@@ -221,14 +221,14 @@
   <link name="gripper_link">
     <visual>
-      <origin xyz="0.0 0.0 0" rpy="0 0 0"/>
-      <geometry>
-        <mesh filename="package://open_manipulator_description/meshes/chain_link_grip_l.stl" scale="0.001 0.001 0.001"/>
-      </geometry>
-      <material name="grey"/>
-    </visual>
-    <collision>
-      <origin xyz="0.0 0.0 0" rpy="0 0 0"/>
-      <geometry>
-        <mesh filename="package://open_manipulator_description/meshes/chain_link_grip_l.stl" scale="0.001 0.001 0.001"/>
+      <origin xyz="0 0 0" rpy="0 0 0"/>
+      <geometry>
+        <mesh filename="package://open_manipulator_description/meshes/chain_link_grip_l.stl"/>
+      </geometry>
+      <material name="grey"/>
+    </visual>
+    <collision>
+      <origin xyz="0 0 0" rpy="0 0 0"/>
+      <geometry>
+        <mesh filename="package://open_manipulator_description/meshes/chain_link_grip_l.stl"/>
       </geometry>
     </collision>
@@ -249,10 +249,10 @@
   </link>
   <!--  Gripper joint -->
-  <joint name="gripper" type="prismatic">
+  <joint name="gripper" type="revolute">
     <parent link="link5"/>
     <child link="gripper_link"/>
-    <origin xyz="0.0817 0.019 0.0" rpy="0 0 0"/>
-    <axis xyz="0 1 0"/>
-    <limit velocity="4.8" effort="1" lower="-0.010" upper="0.019" />
+    <origin xyz="0.04225 0.015 0" rpy="0 0 0"/>
+    <axis xyz="0 0 1"/>
+    <limit velocity="4.8" effort="1" lower="-0.7133010663668231" upper="1.059980724428978" />
   </joint>
   <!-- Transmission 5 -->
@@ -261,14 +261,14 @@
   <link name="gripper_link_sub">
     <visual>
-      <origin xyz="0.0 -0.0 0" rpy="0 0 0"/>
-      <geometry>
-        <mesh filename="package://open_manipulator_description/meshes/chain_link_grip_r.stl" scale="0.001 0.001 0.001"/>
-      </geometry>
-      <material name="grey"/>
-    </visual>
-    <collision>
-      <origin xyz="0.0 -0.0 0" rpy="0 0 0"/>
-      <geometry>
-        <mesh filename="package://open_manipulator_description/meshes/chain_link_grip_r.stl" scale="0.001 0.001 0.001"/>
+      <origin xyz="0 0 0" rpy="0 0 0"/>
+      <geometry>
+        <mesh filename="package://open_manipulator_description/meshes/chain_link_grip_r.stl"/>
+      </geometry>
+      <material name="grey"/>
+    </visual>
+    <collision>
+      <origin xyz="0 0 0" rpy="0 0 0"/>
+      <geometry>
+        <mesh filename="package://open_manipulator_description/meshes/chain_link_grip_r.stl"/>
       </geometry>
     </collision>
@@ -289,11 +289,11 @@
   </link>
   <!--  Gripper joint sub -->
-  <joint name="gripper_sub" type="prismatic">
+  <joint name="gripper_sub" type="revolute">
     <parent link="link5"/>
     <child link="gripper_link_sub"/>
-    <origin xyz="0.0817 -0.019 0" rpy="0 0 0"/>
-    <axis xyz="0 -1 0"/>
-    <limit velocity="4.8" effort="1" lower="-0.010" upper="0.019" />
-    <mimic joint="gripper" multiplier="1"/>
+    <origin xyz="0.04225 -0.015 0" rpy="0 0 0"/>
+    <axis xyz="0 0 1"/>
+    <limit velocity="4.8" effort="1" lower="-0.7133010663668231" upper="1.059980724428978" />
+    <mimic joint="gripper" multiplier="-1"/>
   </joint>
   <!-- Transmission 6 -->

Commit message: Add joint limit and update inertia

File: open_manipulator_description/urdf/open_manipulator.urdf.xacro (robot description, xacro)
@@ -38,15 +38,22 @@
     </visual>
     <collision>
-      <origin xyz="0 0 0" rpy="0 0 0"/>
+      <origin xyz="0 0 0.027" rpy="${-pi/2} 0 0" />
       <geometry>
         <mesh filename="package://open_manipulator_description/meshes/chain_link1.stl" />
       </geometry>
     </collision>
-    <inertial>
-      <origin xyz="-0.016911 -7.3022E-05 -0.0080745" rpy="${-pi/2} 0 0" />
-      <mass value="0.14147" />
-      <inertia ixx="2.1813E-05" ixy="-1.7015E-08" ixz="-8.9152E-07"
-               iyy="2.3447E-05" iyz="-1.5454E-07"
-               izz="1.6364E-06" />
+    <!-- <inertial> -->
+    <!--   <origin xyz="-0.016911 -7.3022E-05 -0.0080745" rpy="${-pi/2} 0 0" /> -->
+    <!--   <mass value="0.14147" /> -->
+    <!--   <inertia ixx="2.1813E-05" ixy="-1.7015E-08" ixz="-8.9152E-07" -->
+    <!--            iyy="2.3447E-05" iyz="-1.5454E-07" -->
+    <!--            izz="1.6364E-06" /> -->
+    <!-- </inertial> -->
+    <inertial>
+      <origin xyz="3.0876154e-04 0.0000000e+00 -1.2176461e-04" />
+      <mass value="7.9119962e-02" />
+      <inertia ixx="1.2505234e-05" ixy="0.0" ixz="-1.7855208e-07"
+               iyy="2.1898364e-05" iyz="0.0"
+               izz="1.9267361e-05" />
     </inertial>
   </link>
@@ -57,5 +64,5 @@
     <origin xyz="0 0 0.0515" rpy="0 0 ${-pi/2}" />
     <axis xyz="0 0 1" />
-    <limit velocity="4.8" effort="1" lower="${-pi}" upper="${pi}" />
+    <limit velocity="4.8" effort="1" lower="${-pi*0.916}" upper="${pi*0.916}" />
   </joint>
   <!-- Transmission 1 -->
@@ -76,10 +83,17 @@
       </geometry>
     </collision>
-    <inertial>
-      <origin xyz="-0.00042334871953208 0.0005762171718733 0.0387383572136045" rpy="0 0 0" />
-      <mass value="0.129397139554481" />
-      <inertia ixx="3.69350041678783E-05" ixy="-3.89313759320941E-08" ixz="-1.11653037527299E-08"
-               iyy="3.68198693987775E-05" iyz="-1.1111795426955E-06"
-               izz="1.48030530212799E-07" />
+    <!-- <inertial> -->
+    <!--   <origin xyz="-0.00042334871953208 0.0005762171718733 0.0387383572136045" rpy="0 0 0" /> -->
+    <!--   <mass value="0.129397139554481" /> -->
+    <!--   <inertia ixx="3.69350041678783E-05" ixy="-3.89313759320941E-08" ixz="-1.11653037527299E-08" -->
+    <!--            iyy="3.68198693987775E-05" iyz="-1.1111795426955E-06" -->
+    <!--            izz="1.48030530212799E-07" /> -->
+    <!-- </inertial> -->
+    <inertial>
+      <origin xyz="-3.0184870e-04 5.4043684e-04 ${0.018 + 2.9433464e-02}" />
+      <mass value="9.8406837e-02" />
+      <inertia ixx="3.4543422e-05" ixy="-1.6031095e-08" ixz="-3.8375155e-07"
+               iyy="3.2689329e-05" iyz="2.8511935e-08"
+               izz="1.8850320e-05" />
     </inertial>
   </link>
@@ -90,5 +104,5 @@
     <origin xyz="0.026 0 0.05475" rpy="${pi/2} 0 ${pi/2}" />
     <axis xyz="0 0 1" />
-    <limit velocity="4.8" effort="1" lower="${-pi}" upper="${pi}" />
+    <limit velocity="4.8" effort="1" lower="${-pi*0.6679}" upper="${pi*0.5965}" />
   </joint>
   <!-- Transmission 2 -->
@@ -109,10 +123,17 @@
       </geometry>
     </collision>
-    <inertial>
-      <origin xyz="0.00634911017847554 0.105401689990389 -0.0262056408085307" rpy="0 0 0" />
-      <mass value="0.12120137926006" />
-      <inertia ixx="0.000489960675623491" ixy="-5.26672832890087E-05" ixz="1.49822052691775E-07"
-               iyy="2.42965312448389E-05" iyz="1.56967790646472E-06"
-               izz="0.000482873776104937" />
+    <!-- <inertial> -->
+    <!--   <origin xyz="0.00634911017847554 0.105401689990389 -0.0262056408085307" rpy="0 0 0" /> -->
+    <!--   <mass value="0.12120137926006" /> -->
+    <!--   <inertia ixx="0.000489960675623491" ixy="-5.26672832890087E-05" ixz="1.49822052691775E-07" -->
+    <!--            iyy="2.42965312448389E-05" iyz="1.56967790646472E-06" -->
+    <!--            izz="0.000482873776104937" /> -->
+    <!-- </inertial> -->
+    <inertial>
+      <origin xyz="1.0308393e-02 3.7743363e-04 1.0170197e-01" />
+      <mass value="1.3850917e-01" />
+      <inertia ixx="3.3055381e-04" ixy="-9.7940978e-08" ixz="-3.8505711e-05"
+               iyy="3.4290447e-04" iyz="-1.5717516e-06"
+               izz="6.0346498e-05" />
     </inertial>
   </link>
@@ -123,5 +144,5 @@
     <origin xyz="0.024 0.1684 -0.045" rpy="0 0 ${pi/2}" />
     <axis xyz="0 0 1" />
-    <limit velocity="4.8" effort="1" lower="${-pi}" upper="${pi}" />
+    <limit velocity="4.8" effort="1" lower="${-pi*0.4611}" upper="${pi*0.5735}" />
   </joint>
   <!-- Transmission 3 -->
@@ -142,10 +163,17 @@
       </geometry>
     </collision>
-    <inertial>
-      <origin xyz="0.0107684769865891 -0.0395998807006063 0.0190000000054333" rpy="0 0 0" />
-      <mass value="0.0597850138451838" />
-      <inertia ixx="1.5907540511103E-05" ixy="2.8291751472122E-06" ixz="-6.22476258071719E-13"
-               iyy="6.16523427095478E-06" iyz="-7.18764926930745E-15"
-               izz="1.15699642937667E-05" />
+    <!-- <inertial> -->
+    <!--   <origin xyz="0.0107684769865891 -0.0395998807006063 0.0190000000054333" rpy="0 0 0" /> -->
+    <!--   <mass value="0.0597850138451838" /> -->
+    <!--   <inertia ixx="1.5907540511103E-05" ixy="2.8291751472122E-06" ixz="-6.22476258071719E-13" -->
+    <!--            iyy="6.16523427095478E-06" iyz="-7.18764926930745E-15" -->
+    <!--            izz="1.15699642937667E-05" /> -->
+    <!-- </inertial> -->
+    <inertial>
+      <origin xyz="9.0909590e-02 3.8929816e-04 2.2413279e-04" />
+      <mass value="1.3274562e-01" />
+      <inertia ixx="3.0654178e-05" ixy="-1.2764155e-06" ixz="-2.6874417e-07"
+               iyy="2.4230292e-04" iyz="1.1559550e-08"
+               izz="2.5155057e-04" />
     </inertial>
   </link>
@@ -156,5 +184,5 @@
     <origin xyz="0 -0.062 0.019" rpy="${pi/2} ${-pi/2} 0" />
     <axis xyz="0 0 1" />
-    <limit velocity="4.8" effort="1" lower="${-pi}" upper="${pi}" />
+    <limit velocity="4.8" effort="1" lower="${-pi*0.994}" upper="${pi*0.994}" />
   </joint>
   <!-- Transmission 4 -->
@@ -175,10 +203,17 @@
       </geometry>
     </collision>
-    <inertial>
-      <origin xyz="-0.000218076760146619 -0.000626191256536957 0.0596980339879584" rpy="0 0 0" />
-      <mass value="0.0796444353162854" />
-      <inertia ixx="6.5346536618451E-05" ixy="1.08804671081198E-08" ixz="3.20425969376465E-07"
-               iyy="6.52473697844542E-05" iyz="1.49110423887788E-06"
-               izz="3.4317718754864E-07" />
+    <!-- <inertial> -->
+    <!--   <origin xyz="-0.000218076760146619 -0.000626191256536957 0.0596980339879584" rpy="0 0 0" /> -->
+    <!--   <mass value="0.0796444353162854" /> -->
+    <!--   <inertia ixx="6.5346536618451E-05" ixy="1.08804671081198E-08" ixz="3.20425969376465E-07" -->
+    <!--            iyy="6.52473697844542E-05" iyz="1.49110423887788E-06" -->
+    <!--            izz="3.4317718754864E-07" /> -->
+    <!-- </inertial> -->
+    <inertial>
+      <origin xyz="4.4206755e-02 3.6839985e-07 8.9142216e-03" />
+      <mass value="1.4327573e-01" />
+      <inertia ixx="8.0870749e-05" ixy="0.0" ixz="-1.0157896e-06"
+               iyy="7.5980465e-05" iyz="0.0"
+               izz="9.3127351e-05" />
     </inertial>
   </link>
@@ -189,5 +224,5 @@
     <origin xyz="0.019 0 0.088" rpy="${pi/2} 0 ${pi/2}" />
     <axis xyz="0 0 1" />
-    <limit velocity="4.8" effort="1" lower="${-pi}" upper="${pi}" />
+    <limit velocity="4.8" effort="1" lower="${-pi*0.7073}" upper="${pi*0.5735}" />
   </joint>
   <!-- Transmission 5 -->
@@ -208,10 +243,17 @@
       </geometry>
     </collision>
-    <inertial>
-      <origin xyz="-0.0107684769865891 0.0395998807006062 -0.0189999999945667" rpy="0 0 0" />
-      <mass value="0.0597850138451838" />
-      <inertia ixx="1.59075405111031E-05" ixy="2.8291751472122E-06" ixz="6.22476246848532E-13"
-               iyy="6.16523427095479E-06" iyz="7.18764844874428E-15"
-               izz="1.15699642937667E-05" />
+    <!-- <inertial> -->
+    <!--   <origin xyz="-0.0107684769865891 0.0395998807006062 -0.0189999999945667" rpy="0 0 0" /> -->
+    <!--   <mass value="0.0597850138451838" /> -->
+    <!--   <inertia ixx="1.59075405111031E-05" ixy="2.8291751472122E-06" ixz="6.22476246848532E-13" -->
+    <!--            iyy="6.16523427095479E-06" iyz="7.18764844874428E-15" -->
+    <!--            izz="1.15699642937667E-05" /> -->
+    <!-- </inertial> -->
+    <inertial>
+      <origin xyz="4.4206755e-02 3.6839985e-07 8.9142216e-03" />
+      <mass value="1.4327573e-01" />
+      <inertia ixx="8.0870749e-05" ixy="0.0" ixz="-1.0157896e-06"
+               iyy="7.5980465e-05" iyz="0.0"
+               izz="9.3127351e-05" />
     </inertial>
   </link>
@@ -222,5 +264,5 @@
     <origin xyz="0 0.062 -0.019" rpy="${-pi/2} 0 ${pi}" />
     <axis xyz="0 0 1" />
-    <limit velocity="4.8" effort="1" lower="${-pi}" upper="${pi}" />
+    <limit velocity="4.8" effort="1" lower="${-pi*0.994}" upper="${pi*0.994}" />
   </joint>
   <!-- Transmission 6 -->
@@ -241,11 +283,18 @@
       </geometry>
     </collision>
-    <inertial>
-      <origin xyz="8.11464269925566E-05 -0.00070824109768956 -0.0220980053972996" rpy="0 0 0" />
-      <mass value="0.0741805648173052" />
-      <inertia ixx="5.00300817099651E-06" ixy="-2.1246207546751E-07" ixz="2.45442201688391E-08"
-               iyy="9.69324841658574E-06" iyz="-2.18474747851751E-06"
-               izz="8.88278852334281E-06" />
-    </inertial>
+    <!-- <inertial> -->
+    <!--   <origin xyz="8.11464269925566E-05 -0.00070824109768956 -0.0220980053972996" rpy="0 0 0" /> -->
+    <!--   <mass value="0.0741805648173052" /> -->
+    <!--   <inertia ixx="5.00300817099651E-06" ixy="-2.1246207546751E-07" ixz="2.45442201688391E-08" -->
+    <!--            iyy="9.69324841658574E-06" iyz="-2.18474747851751E-06" -->
+    <!--            izz="8.88278852334281E-06" /> -->
+    <!-- </inertial> -->
+         <inertial>
+           <origin xyz="4.4206755e-02 3.6839985e-07 8.9142216e-03" />
+           <mass value="1.4327573e-01" />
+           <inertia ixx="8.0870749e-05" ixy="0.0" ixz="-1.0157896e-06"
+                    iyy="7.5980465e-05" iyz="0.0"
+                    izz="9.3127351e-05" />
+         </inertial>
   </link>
   <!--  Gripper link -->
@@ -278,5 +327,5 @@
     <origin xyz="0.027 -0.016 -0.026" rpy="${-pi/2} ${pi/4} ${-pi/2}" />
     <axis xyz="0 0 1" />
-    <limit velocity="4.8" effort="1" lower="${-pi}" upper="${pi}" />
+    <limit velocity="4.8" effort="1" lower="-0.7133010663668231" upper="1.059980724428978" />
   </joint>
   <!-- Transmission 7 -->
@@ -311,5 +360,6 @@
     <origin xyz="0.027 0.016 -0.026" rpy="${-pi/2} ${pi/4} ${-pi/2}" />
     <axis xyz="0 0 1" />
-    <limit velocity="4.8" effort="1" lower="${-pi}" upper="${pi}" />
+    <limit velocity="4.8" effort="1" lower="-0.7133010663668231" upper="1.059980724428978" />
+    <!-- <limit velocity="4.8" effort="1" lower="${-pi*0.250}" upper="${pi*0.5777}" /> -->
     <mimic joint="gripper" multiplier="-1"/>
   </joint>
