Commit message: Fix joint coordinates

File: open_manipulator_description/urdf/open_manipulator.urdf.xacro (robot description, xacro)
@@ -62,5 +62,5 @@
     <parent link="link1" />
     <child link="link2" />
-    <origin xyz="0 0 0.0515" rpy="0 0 ${-pi/2}" />
+    <origin xyz="0 0 0.0515" rpy="0 0 0" />
     <axis xyz="0 0 1" />
     <limit velocity="4.8" effort="1" lower="${-pi*0.916}" upper="${pi*0.916}" />
@@ -71,5 +71,5 @@
   <link name="link2">
     <visual>
-      <origin xyz="0 0 0" rpy="0 0 0" />
+      <origin xyz="0 0 0" rpy="0 0 ${-pi/2}" />
       <geometry>
         <mesh filename="package://open_manipulator_description/meshes/chain_link2.stl" />
@@ -78,5 +78,5 @@
     </visual>
     <collision>
-      <origin xyz="0 0 0" rpy="0 0 0" />
+      <origin xyz="0 0 0" rpy="0 0 ${pi/2}" />
       <geometry>
         <mesh filename="package://open_manipulator_description/meshes/chain_link2.stl" />
@@ -102,6 +102,6 @@
     <parent link="link2" />
     <child link="link3" />
-    <origin xyz="0.026 0 0.05475" rpy="${pi/2} 0 ${pi/2}" />
-    <axis xyz="0 0 1" />
+    <origin xyz="0 0 0.05475" rpy="0 0 0" />
+    <axis xyz="0 1 0" />
     <limit velocity="4.8" effort="1" lower="${-pi*0.6679}" upper="${pi*0.5965}" />
   </joint>
@@ -111,5 +111,5 @@
   <link name="link3">
     <visual>
-      <origin xyz="0 0 0" rpy="0 0 0" />
+      <origin xyz="0 -0.026 0" rpy="${pi/2} 0 0" />
       <geometry>
         <mesh filename="package://open_manipulator_description/meshes/chain_link3.stl" />
@@ -118,5 +118,5 @@
     </visual>
     <collision>
-      <origin xyz="0 0 0" rpy="0 0 0" />
+      <origin xyz="0 -0.026 0" rpy="${pi/2} 0 0" />
       <geometry>
         <mesh filename="package://open_manipulator_description/meshes/chain_link3.stl" />
@@ -142,7 +142,7 @@
     <parent link="link3" />
     <child link="link4" />
-    <origin xyz="0.024 0.1684 -0.045" rpy="0 0 ${pi/2}" />
-    <axis xyz="0 0 1" />
-    <limit velocity="4.8" effort="1" lower="${-pi*0.4611}" upper="${pi*0.5735}" />
+    <origin xyz="0.024 0 0.1684" rpy="0 0 0" />
+    <axis xyz="0 1 0" />
+    <limit velocity="4.8" effort="1" lower="${-pi*0.5735}" upper="${pi*0.448}" />
   </joint>
   <!-- Transmission 3 -->
@@ -151,5 +151,5 @@
   <link name="link4">
     <visual>
-      <origin xyz="0 0 0" rpy="0 0 0" />
+      <origin xyz="0 0.019 0" rpy="${pi/2} ${-pi/2} 0" />
       <geometry>
         <mesh filename="package://open_manipulator_description/meshes/chain_link4.stl" />
@@ -158,5 +158,5 @@
     </visual>
     <collision>
-      <origin xyz="0 0 0" rpy="0 0 0" />
+      <origin xyz="0 0.019 0" rpy="${pi/2} ${-pi/2} 0" />
       <geometry>
         <mesh filename="package://open_manipulator_description/meshes/chain_link4.stl" />
@@ -182,6 +182,6 @@
     <parent link="link4" />
     <child link="link5" />
-    <origin xyz="0 -0.062 0.019" rpy="${pi/2} ${-pi/2} 0" />
-    <axis xyz="0 0 1" />
+    <origin xyz="0.062 0 0" rpy="0 0 0" />
+    <axis xyz="1 0 0" />
     <limit velocity="4.8" effort="1" lower="${-pi*0.994}" upper="${pi*0.994}" />
   </joint>
@@ -191,5 +191,5 @@
   <link name="link5">
     <visual>
-      <origin xyz="0 0 0" rpy="0 0 0" />
+      <origin xyz="0 0 0" rpy="${pi/2} ${pi} ${pi/2}" />
       <geometry>
         <mesh filename="package://open_manipulator_description/meshes/chain_link5.stl" />
@@ -198,5 +198,5 @@
     </visual>
     <collision>
-      <origin xyz="0 0 0" rpy="0 0 0" />
+      <origin xyz="0 0 0" rpy="${pi/2} ${pi} ${pi/2}" />
       <geometry>
         <mesh filename="package://open_manipulator_description/meshes/chain_link5.stl" />
@@ -222,7 +222,7 @@
     <parent link="link5" />
     <child link="link6" />
-    <origin xyz="0.019 0 0.088" rpy="${pi/2} 0 ${pi/2}" />
-    <axis xyz="0 0 1" />
-    <limit velocity="4.8" effort="1" lower="${-pi*0.7073}" upper="${pi*0.5735}" />
+    <origin xyz="0.088 0 0" rpy="0 0 0" />
+    <axis xyz="0 1 0" />
+    <limit velocity="4.8" effort="1" lower="${-pi*0.5735}" upper="${pi*0.7073}" />
   </joint>
   <!-- Transmission 5 -->
@@ -231,5 +231,5 @@
   <link name="link6">
     <visual>
-      <origin xyz="0 0 0" rpy="0 0 0" />
+      <origin xyz="0 -0.019 0" rpy="${pi/2} ${pi/2} 0" />
       <geometry>
         <mesh filename="package://open_manipulator_description/meshes/chain_link6.stl" />
@@ -238,5 +238,5 @@
     </visual>
     <collision>
-      <origin xyz="0 0 0" rpy="0 0 0" />
+      <origin xyz="0 -0.019 0" rpy="${pi/2} ${pi/2} 0" />
       <geometry>
         <mesh filename="package://open_manipulator_description/meshes/chain_link6.stl" />
@@ -262,6 +262,6 @@
     <parent link="link6" />
     <child link="link7" />
-    <origin xyz="0 0.062 -0.019" rpy="${-pi/2} 0 ${pi}" />
-    <axis xyz="0 0 1" />
+    <origin xyz="0.062 0 0" rpy="0 0 0" />
+    <axis xyz="1 0 0" />
     <limit velocity="4.8" effort="1" lower="${-pi*0.994}" upper="${pi*0.994}" />
   </joint>
@@ -271,5 +271,5 @@
   <link name="link7">
     <visual>
-      <origin xyz="0 0 0" rpy="0 0 0" />
+      <origin xyz="0 0 0" rpy="0 ${-pi/2} 0" />
       <geometry>
         <mesh filename="package://open_manipulator_description/meshes/chain_link7.stl" />
@@ -278,5 +278,5 @@
     </visual>
     <collision>
-      <origin xyz="0 0 0" rpy="0 0 0" />
+      <origin xyz="0 0 0" rpy="0 ${-pi/2} 0" />
       <geometry>
         <mesh filename="package://open_manipulator_description/meshes/chain_link7.stl" />
@@ -301,5 +301,38 @@
   <link name="gripper_link">
     <visual>
-      <origin xyz="0 0 -0.027" rpy="0 0 0" />
+      <origin xyz="0 0 0" rpy="0 0 0" />
+      <geometry>
+        <mesh filename="package://open_manipulator_description/meshes/chain_link_grip_l.stl" />
+      </geometry>
+      <material name="grey"/>
+    </visual>
+    <collision>
+      <origin xyz="0 0 0" rpy="0 0 0" />
+      <geometry>
+        <mesh filename="package://open_manipulator_description/meshes/chain_link_grip_l.stl" />
+      </geometry>
+    </collision>
+    <inertial>
+      <origin xyz="-0.00340216508542759 -0.00576540023107835 -2.1799589910998E-09" rpy="0 0 0" />
+      <mass value="0.0356307403873285" />
+      <inertia ixx="1.81811062489467E-05" ixy="2.51217685396069E-06" ixz="-1.0866660092931E-08"
+               iyy="9.13797195647898E-06" iyz="-1.08688133683192E-08"
+               izz="1.03452048539682E-05" />
+    </inertial>
+  </link>
+  <!--  Gripper joint -->
+  <joint name="gripper" type="revolute">
+    <parent link="link7" />
+    <child link="gripper_link" />
+    <origin xyz="0.026 0.016 0" rpy="0 0 0" />
+    <axis xyz="0 0 1" />
+    <limit velocity="4.8" effort="1" lower="-0.7133010663668231" upper="1.059980724428978" />
+  </joint>
+  <!-- Transmission 7 -->
+  <xacro:SimpleTransmission n="7" joint="gripper" />
+  <!--  Gripper link sub-->
+  <link name="gripper_link_sub">
+    <visual>
+      <origin xyz="0 0 0" rpy="0 0 0" />
       <geometry>
         <mesh filename="package://open_manipulator_description/meshes/chain_link_grip_r.stl" />
@@ -308,5 +341,5 @@
     </visual>
     <collision>
-      <origin xyz="0 0 -0.027" rpy="0 0 0" />
+      <origin xyz="0 0 0" rpy="0 0 0" />
       <geometry>
         <mesh filename="package://open_manipulator_description/meshes/chain_link_grip_r.stl" />
@@ -321,45 +354,11 @@
     </inertial>
   </link>
-  <!--  Gripper joint -->
-  <joint name="gripper" type="revolute">
-    <parent link="link7" />
-    <child link="gripper_link" />
-    <origin xyz="0.027 -0.016 -0.026" rpy="${-pi/2} ${pi/4} ${-pi/2}" />
-    <axis xyz="0 0 1" />
-    <limit velocity="4.8" effort="1" lower="-0.7133010663668231" upper="1.059980724428978" />
-  </joint>
-  <!-- Transmission 7 -->
-  <xacro:SimpleTransmission n="7" joint="gripper" />
-  <!--  Gripper link sub -->
-  <link name="gripper_link_sub">
-    <visual>
-      <origin xyz="0 0 -0.027" rpy="0 0 ${pi/2}" />
-      <geometry>
-        <mesh filename="package://open_manipulator_description/meshes/chain_link_grip_l.stl" />
-      </geometry>
-      <material name="grey"/>
-    </visual>
-    <collision>
-      <origin xyz="0 0 -0.027" rpy="0 0 ${pi/2}" />
-      <geometry>
-        <mesh filename="package://open_manipulator_description/meshes/chain_link_grip_l.stl" />
-      </geometry>
-    </collision>
-    <inertial>
-      <origin xyz="-0.00340216508542759 -0.00576540023107835 -2.1799589910998E-09" rpy="0 0 0" />
-      <mass value="0.0356307403873285" />
-      <inertia ixx="1.81811062489467E-05" ixy="2.51217685396069E-06" ixz="-1.0866660092931E-08"
-               iyy="9.13797195647898E-06" iyz="-1.08688133683192E-08"
-               izz="1.03452048539682E-05" />
-    </inertial>
-  </link>
   <!--  Gripper joint sub -->
   <joint name="gripper_sub" type="revolute">
     <parent link="link7" />
     <child link="gripper_link_sub" />
-    <origin xyz="0.027 0.016 -0.026" rpy="${-pi/2} ${pi/4} ${-pi/2}" />
+    <origin xyz="0.026 -0.016 0" rpy="0 0 0" />
     <axis xyz="0 0 1" />
     <limit velocity="4.8" effort="1" lower="-0.7133010663668231" upper="1.059980724428978" />
-    <!-- <limit velocity="4.8" effort="1" lower="${-pi*0.250}" upper="${pi*0.5777}" /> -->
     <mimic joint="gripper" multiplier="-1"/>
   </joint>
@@ -368,5 +367,5 @@
   <!-- end effector joint -->
   <joint name="end_effector_joint" type="fixed">
-    <origin xyz="0.0 0.0 -0.086" rpy="0 0 0"/>
+    <origin xyz="0.08375 0 0" rpy="0 0 0"/>
     <parent link="link7"/>
     <child link="end_effector_link"/>
@@ -382,5 +381,5 @@
      </visual>
     <inertial>
-      <origin xyz="0.0 0.0 0.0" rpy="0 0 0"/>
+      <origin xyz="0 0 0" rpy="0 0 0"/>
       <mass value="0.001"/>
       <inertia ixx="1.0e-06" ixy="0.0" ixz="0.0" iyy="1.0e-06" iyz="0.0" izz="1.0e-06" />
